File: RasPi-BplusHAT_CamSlot.brd (EAGLE design)
At the start: 65 x 56 mm, 66 parts, among them IC1 MAX31855, IC2 MAX31855, IC3 MAX31855, J1 1X2-3.5MM, J2 1X2-3.5MM, J3 1X2-3.5MM, J7 4P-2.0, J8 4P-2.0, K1 PIN20X2, Q1 NFET-FDD8780, U1 EEPROM24, U2 ATMEGA328P

Commit message: wip
Parts:
- removed C13: 47uF, SparkFun-Capacitors:PANASONIC_D
- removed TEMP: (no value), SparkFun-Connectors:MOLEX-1X4_LOCK
- added C14: 0.1uF, SparkFun-Passives:0805
- added JP1: (no value), SparkFun-Connectors:MOLEX-1X3
- added SJ1, SJ2: (no value), SparkFun-Retired:SJ_3
- added TP4, TP5, TP6, TP8: 3V3, SparkFun-Passives:TP_15TH
- added TP7: GND, SparkFun-Passives:PAD.03X.04
- added Y1: 8MHZ, SparkFun-FreqCtrl:RESONATOR-SMD
- C1: value 100nF -> 47uF; device resistor:C0805K -> SparkFun-Capacitors:EIA7343
- C12, C7: value 10UF-25V -> 47uF; device SparkFun-Capacitors:EIA6032-NOM -> SparkFun-Capacitors:EIA7343
- JP2: device SparkFun-Connectors:JST-2-PTH-VERT -> SparkFun-Connectors:MOLEX-1X2_LOCK
- R1, R2: value 3k9 -> 10K; device resistor:M0805 -> SparkFun-Resistors:0603-RES
- R10, R11: value 10K -> 100K
- R3: value 1k -> 10K; device resistor:M0805 -> SparkFun-Resistors:0603-RES
- moved TP2 57.0 mm to (58.5, 7.62)
- moved TP3 51.3 mm to (47.6, 36.4)
- moved ATRST 37.0 mm to (60.0, 31.9)
- moved C1 27.1 mm to (40.1, 15.2), turned to 90 degrees
- moved R12 24.3 mm to (30.5, 30.0), flipped to the bottom, turned to 270 degrees
- moved C6 21.0 mm to (26.0, 38.4), flipped to the bottom
- moved LOGO1 20.1 mm to (46.5, 25.9)
- moved R4 17.2 mm to (26.0, 29.9), flipped to the bottom, turned to 270 degrees
- moved R9 15.9 mm to (20.4, 29.0), flipped to the bottom, turned to 0 degrees
- moved U2 15.8 mm to (27.4, 37.8)
- moved R11 15.3 mm to (14.4, 30.0)
- moved R3 12.3 mm to (51.5, 44.0), flipped to the bottom
- moved C5 12.2 mm to (29.0, 38.2), flipped to the bottom, turned to 90 degrees
- moved R10 11.5 mm to (14.5, 35.8), turned to 270 degrees
- moved C8 10.5 mm to (20.6, 32.8), flipped to the bottom, turned to 0 degrees
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Connections:
- removed net VCC: IC1.4, IC2.4, IC3.4, J7.3, J8.3
- new net N$25: Q1.1, SJ2.2
- new net N$26: U2.7, Y1.1
- new net N$27: U2.8, Y1.3
- new net N$28: JP1.1
- new net PD5: SJ2.1
- net +3V3: now also C14.1, TP4.P$1; no longer C1.1, K1.1, K1.17
- net +5V: now also C7.A, TP6.P$1; no longer C13.+
- net 12V: now also C1.A, TP5.P$1; no longer C7.A
- net 3.3V: now also IC1.4, IC2.4, IC3.4, J7.3, J8.3, K1.1, K1.17
- net ADC0: now also JP1.3, R11.1; no longer TEMP.3
- net ADC1: now also JP1.2, R10.1; no longer TEMP.1
- net GND: now also C1.C, C14.2, TP7.P$1, TP8.P$1, Y1.2; no longer C1.2, C13.-, JP10.1
- net N$16: now also JP2.2, SJ1.3; no longer R11.1, TEMP.4
- net N$17: now also JP10.1, SJ1.1; no longer R10.1, TEMP.2
- net N$22: now also SJ1.2; no longer JP2.2
- net PWM: now also SJ2.3; no longer Q1.1
Routing:
- net +3V3: track 140.1 -> 0.00 mm, vias 4 -> 0
- net 12V: track 122.3 -> 0.00 mm
- net +5V: track 119.4 -> 0.00 mm
- net ATRST: track 85.8 -> 0.00 mm, vias 4 -> 0
- net LED1: track 77.8 -> 0.00 mm, vias 4 -> 0
- net ATMOSI: track 72.4 -> 0.00 mm, vias 1 -> 0
- net ATSCK: track 72.0 -> 0.00 mm, vias 1 -> 0
- net SENSE: track 69.3 -> 0.00 mm, vias 2 -> 0
- net AT5: track 69.0 -> 0.00 mm, vias 2 -> 0
- net ATMISO: track 62.7 -> 0.00 mm, vias 2 -> 0
- net SDA: track 58.3 -> 0.00 mm, vias 1 -> 0
- net CS0: track 56.8 -> 0.00 mm, vias 2 -> 0
- net VCC: track 55.6 -> 0.00 mm
- net SCLK: track 54.5 -> 0.00 mm, vias 2 -> 0
- net LED3: track 53.3 -> 0.00 mm
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
Commit message: as sent to oshpark for rev2
Parts:
- removed R14, R15, R16: 330, SparkFun-Resistors:0603-RES
- added PWR: (no value), SparkFun-LED:LED-0603
- added R17: 330, SparkFun-Resistors:0603-ARV
- JP1: device SparkFun-Connectors:MOLEX-1X3 -> SparkFun-Connectors:SCREWTERMINAL-3.5MM-3
- moved C8 42.5 mm to (62.9, 37.8), flipped to the top, turned to 90 degrees
- moved C12 28.6 mm to (51.9, 4.25), turned to 180 degrees
- moved C7 28.6 mm to (52.1, 32.8), turned to 90 degrees
- moved R12 26.5 mm to (5.62, 39.1), flipped to the top, turned to 0 degrees
- moved R9 13.6 mm to (24.6, 41.9), flipped to the top, turned to 180 degrees
- moved R4 12.6 mm to (29.8, 41.9), flipped to the top, turned to 180 degrees
- moved Y1 7.31 mm to (22.2, 29.5), turned to 0 degrees
- moved C6 6.47 mm to (21.1, 34.1), flipped to the top, turned to 90 degrees
- moved C5 4.98 mm to (33.8, 39.8), flipped to the top, turned to 270 degrees
- moved SJ1 4.30 mm to (56.5, 11.0)
- moved D1 4.16 mm to (17.5, 39.0)
- moved U2 3.61 mm to (28.2, 34.2)
- moved R13 3.02 mm to (19.9, 39.1)
- moved TP7 2.47 mm to (3.75, 8.50)
- moved R10 2.03 mm to (16.5, 35.4)
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Connections:
- removed net 3.3V: C10.1, C11.1, C9.1, IC1.4, IC2.4, IC3.4, J7.3, J8.3, K1.1, K1.17, R10.2, R11.2
- removed net N$28: JP1.1
- new net PWR: PWR.C, R17.5
- net +3V3: now also C10.1, C11.1, C9.1, IC1.4, IC2.4, IC3.4, J7.3, J8.3, K1.1, K1.17, PWR.A, R10.2, R11.2; no longer R12.2
- net AT5: now also R12.2
- net GND: now also JP1.1, R17.1, R17.2, R17.3, R17.4; no longer R14.1, R15.1, R16.1
- net N$21: now also R17.8; no longer R14.2
- net N$23: now also R17.7; no longer R15.2
- net N$24: now also R17.6; no longer R16.2
- net PD5: now also U2.9
Routing:
- net +3V3: track 0.00 -> 154.6 mm
- net ATRST: track 0.00 -> 108.8 mm, vias 0 -> 2
- net ATMISO: track 0.00 -> 94.2 mm, vias 0 -> 1
- net SCLK: track 0.00 -> 94.2 mm, vias 0 -> 2
- net ATSCK: track 0.00 -> 85.2 mm, vias 0 -> 4
- net SENSE: track 0.00 -> 83.8 mm, vias 0 -> 4
- net CS1: track 0.00 -> 78.2 mm, vias 0 -> 2
- net 12V: track 0.00 -> 78.1 mm
- net ATMOSI: track 0.00 -> 70.8 mm, vias 0 -> 5
- net SCL: track 0.00 -> 68.6 mm, vias 0 -> 1
- net MISO: track 0.00 -> 65.9 mm, vias 0 -> 5
- net LED3: track 0.00 -> 64.5 mm, vias 0 -> 1
- net LED1: track 0.00 -> 63.0 mm
- net N$19: track 0.00 -> 62.6 mm, vias 0 -> 2
- net CS0: track 0.00 -> 62.5 mm, vias 0 -> 4
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Other:
- board text added: "2-WIRE"
- board text added: "4-WIRE"
- board text added: "ADC0"
- board text added: "ADC1"
- board text added: "Robosmoker"
- board text added: "https://github.com/robosmoker"
