File: RasPi-BplusHAT_CamSlot.sch (EAGLE design)
At the start: 66 parts, among them IC1 MAX31855, IC2 MAX31855, IC3 MAX31855, J1 1X2-3.5MM, J2 1X2-3.5MM, J3 1X2-3.5MM, J7 4P-2.0, J8 4P-2.0, K1 PIN20X2, Q1 NFET-FDD8780, U1 EEPROM24, U2 ATMEGA328P

Commit message: some fixmes
Other:
- note added: "FIXME: consistent size and value of resistors"
- note added: "FIXME: mark pin 1 better"
- note added: "FIXME: mark polarity of conn in silk"
- note added: "FIXME: pullup to at5"
- note added: "FIXME: silk polarity backwards"
Changed lines of the file:
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@@
 <text x="293.37" y="124.46" size="1.778" layer="91">For fan ctrl, see
 http://www.formfactors.org/developer/specs/REV1_2_Public.pdf</text>
+<text x="128.27" y="97.79" size="1.778" layer="91">FIXME: pullup to at5</text>
+<text x="273.05" y="125.73" size="1.778" layer="91" rot="R90">FIXME: silk polarity backwards</text>
+<text x="41.91" y="200.66" size="1.778" layer="91">FIXME: mark pin 1 better</text>
+<text x="67.31" y="233.68" size="1.778" layer="91">FIXME: consistent size and value of resistors</text>
+<text x="160.02" y="144.78" size="1.778" layer="91">FIXME: mark polarity of conn in silk</text>
 </plain>
 <instances>

Commit message: wip
Parts:
- removed C13: 47uF, SparkFun-Capacitors:47UF-50V-20%(ELECT)
- removed TEMP: (no value), SparkFun-Connectors:M04POLAR_LOCK
- added C14: 0.1uF, SparkFun-Passives:CAP0805
- added JP1: (no value), SparkFun-Connectors:M03POLAR
- added SJ1, SJ2: (no value), SparkFun-Retired:SOLDERJUMPER_2WAYS
- added TP4, TP5, TP6, TP8: 3V3, SparkFun-Passives:TEST-POINTTP_15TH_THRU
- added TP7: GND, SparkFun-Passives:TEST-POINT3X4
- added Y1: 8MHZ, SparkFun-FreqCtrl:RESONATOR8MHZ
- C1: value 100nF -> 47uF; device resistor:C-EUC0805K -> SparkFun-Capacitors:CAP_POL7343; DIELECTRIC X7R -> (none)
- C12, C7: value 10UF-25V -> 47uF; device SparkFun-Capacitors:10UF-25V-10%(SMT-TANT) -> SparkFun-Capacitors:CAP_POL7343
- JP2: device SparkFun-Connectors:M02JST-PTH-VERT -> SparkFun-Connectors:M02POLAR_LOCK
- R1, R2: value 3k9 -> 10K; device resistor:R-EU_M0805 -> SparkFun-Resistors:10KOHM-1/10W-1%(0603)0603; TOLERANCE 5% -> (none)
- R10, R11: value 10K -> 100K
- R3: value 1k -> 10K; device resistor:R-EU_M0805 -> SparkFun-Resistors:10KOHM-1/10W-1%(0603)0603; TOLERANCE 5% -> (none)
Connections:
- removed net VCC: IC1.VCC, IC2.VCC, IC3.VCC, J7.3, J8.3
- new net N$25: Q1.G, SJ2.2
- new net N$26: U2.PB6(XTAL1/TOSC1), Y1.1
- new net N$27: U2.PB7(XTAL2/TOSC2), Y1.3
- new net N$28: JP1.1
- new net PD5: SJ2.1
- net +3V3: now also C14.1, TP4.1; no longer C1.1, K1.1, K1.17
- net +5V: now also C7.+, TP6.1; no longer C13.+
- net 12V: now also C1.+, TP5.1; no longer C7.+
- net 3.3V: now also IC1.VCC, IC2.VCC, IC3.VCC, J7.3, J8.3, K1.1, K1.17
- net ADC0: now also JP1.3, R11.1; no longer TEMP.3
- net ADC1: now also JP1.2, R10.1; no longer TEMP.1
- net GND: now also C1.-, C14.2, TP7.1, TP8.1, Y1.2; no longer C1.2, C13.-, JP10.1
- net N$16: now also JP2.2, SJ1.3; no longer R11.1, TEMP.4
- net N$17: now also JP10.1, SJ1.1; no longer R10.1, TEMP.2
- net N$22: now also SJ1.2; no longer JP2.2
- net PWM: now also SJ2.3; no longer Q1.G
Other:
- note removed: "FIXME: consistent size and value of resistors"
- note removed: "FIXME: silk polarity backwards"
- moved on the sheet: C12, C7, D2, D3, JP2, Q1, R10, R8, TP2, TP3

Commit message: as sent to oshpark for rev2
Parts:
- removed R14, R15, R16: 330, SparkFun-Resistors:RESISTOR0603
- added PWR: (no value), SparkFun-LED:LED0603
- added R17: 330, SparkFun-Resistors:RESISTOR-ARRAY0603-ARV
- JP1: device SparkFun-Connectors:M03POLAR -> SparkFun-Connectors:M03SCREW
Connections:
- removed net 3.3V: C10.1, C11.1, C9.1, IC1.VCC, IC2.VCC, IC3.VCC, J7.3, J8.3, K1.1, K1.17, R10.2, R11.2
- removed net N$28: JP1.1
- new net PWR: PWR.C, R17D.2
- net +3V3: now also C10.1, C11.1, C9.1, IC1.VCC, IC2.VCC, IC3.VCC, J7.3, J8.3, K1.1, K1.17, PWR.A, R10.2, R11.2; no longer R12.2
- net AT5: now also R12.2
- net GND: now also JP1.1, R17A.1, R17B.1, R17D.1, R17R.1; no longer R14.1, R15.1, R16.1
- net N$21: now also R17A.2; no longer R14.2
- net N$23: now also R17B.2; no longer R15.2
- net N$24: now also R17R.2; no longer R16.2
- net PD5: now also U2.PD5(T1)
Other:
- note removed: "FIXME: mark polarity of conn in silk"
- note removed: "FIXME: pullup to at5"
- moved on the sheet: JP1
