File: robosmoker.sch (EAGLE design)
At the start: 73 parts, among them IC1 MAX31855, IC2 MAX31855, IC3 MAX31855, J1 1X2-3.5MM, J2 1X2-3.5MM, J3 1X2-3.5MM, J7 4P-2.0, J8 4P-2.0, K1 PIN20X2, Q1 NFET-FDD8780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

Commit message: tidying up things
Other:
- note added: "Michael Leibowitz"
- note added: "v2.1"
- note removed: "FLYFISH TECHNOLOGIES d.o.o."
- note removed: "Ivan Zilic"
- note removed: "v0.1"
Changed lines of the file:
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@@
 <setting verticaltext="up"/>
 </settings>
-<grid distance="0.05" unitdist="inch" unit="inch" style="lines" multiple="1" display="no" altdistance="0.01" altunitdist="inch" altunit="inch"/>
+<grid distance="0.1" unitdist="inch" unit="inch" style="lines" multiple="1" display="no" altdistance="0.01" altunitdist="inch" altunit="inch"/>
 <layers>
 <layer number="1" name="Top" color="4" fill="1" visible="no" active="no"/>
@@
 </layers>
 <schematic xreflabel="%F%N/%S.%C%R" xrefpart="/%S.%C%R">
+<description>http://github.com/robosmoker</description>
 <attributes>
 </attributes>
@@
 <text x="289.56" y="20.32" size="1.778" layer="94" ratio="15">Drawn by:</text>
 <text x="289.56" y="16.51" size="1.778" layer="94" ratio="15">Checked  by:</text>
-<text x="289.56" y="5.08" size="1.778" layer="94">FLYFISH TECHNOLOGIES d.o.o.</text>
-<text x="309.88" y="20.32" size="1.778" layer="94">Ivan Zilic</text>
-<text x="374.65" y="5.08" size="2.54" layer="94" ratio="10">v0.1</text>
+<text x="309.88" y="20.32" size="1.778" layer="94">Michael Leibowitz</text>
+<text x="374.65" y="5.08" size="2.54" layer="94" ratio="10">v2.1</text>
 <text x="293.37" y="124.46" size="1.778" layer="91">For fan ctrl, see
 http://www.formfactors.org/developer/specs/REV1_2_Public.pdf</text>
